Commit message: Finished refactoring

File: body.urdf (robot description, URDF)
Before this commit: robot robot, 3 links, 2 joints
Joints:
- joint Torso_FrontLeg: origin xyz=-0.5 0 1 rpy=0 0 0 -> xyz=1.5 0 1 rpy=0 0 0

Commit message: Milestone 1

File: body.urdf (robot description, URDF)
Before this commit: robot robot, 9 links, 8 joints
Links:
- removed link BackLeg
- removed link BackLowerLeg
- removed link FrontLeg
- removed link FrontLowerLeg
- removed link LeftLowerLeg
- removed link RightLowerLeg
- added link LeftArm, mass 1; collision box size=0.5 0.25 0.75; visual box size=0.5 0.25 0.75
- added link RightArm, mass 1; collision box size=0.5 0.25 0.75; visual box size=0.5 0.25 0.75
- link LeftLeg: geometry collision box size=0.5 0.5 1.5; visual box size=0.5 0.5 1.5
- link RightLeg: geometry collision box size=0.5 0.5 1.5; visual box size=0.5 0.5 1.5
- link Torso: geometry collision box size=1 0.5 1.25; visual box size=1 0.5 1.25
Joints:
- removed joint BackLeg_BackLowerLeg
- removed joint FrontLeg_FrontLowerLeg
- removed joint LeftLeg_LeftLowerLeg
- removed joint RightLeg_RightLowerLeg
- removed joint Torso_BackLeg
- removed joint Torso_FrontLeg
- added joint Torso_LeftArm: type revolute, parent Torso, child LeftArm, origin xyz=0.5 0 2.875 rpy=0 0 0, axis 0 1 0, limit lower=-3.14159 upper=3.14159 effort=0.0 velocity=0.0
- added joint Torso_RightArm: type revolute, parent Torso, child RightArm, origin xyz=1.5 0 2.875 rpy=0 0 0, axis 0 1 0, limit lower=-3.14159 upper=3.14159 effort=0.0 velocity=0.0
- joint Torso_LeftLeg: axis 0 1 0 -> 1 0 0; origin xyz=-0.5 0 1 rpy=0 0 0 -> xyz=0.75 0 1.89 rpy=0 0 0
- joint Torso_RightLeg: axis 0 1 0 -> 1 0 0; origin xyz=0.5 0 1 rpy=0 0 0 -> xyz=1.25 0 1.89 rpy=0 0 0
